File: PCB/Suboscillator.kicad_pcb (KiCad board)
At the start: 2 copper layers, 45 x 58 mm, 33 parts, among them J1 Conn_01x02 Osc In, J2 EURO_PWR_2x5, J3 Conn_01x03, J4 Conn_01x02 Sub Osc Out, J5 Conn_01x02 Sub Osc Out, J6 Conn_01x02 Sub Osc Out, J7 Conn_01x01, J8 Conn_01x01, Q1 BC547, U1 4013

Commit message: Add panel components
Parts:
- J1: value Conn_01x02 Osc In -> Molex_KK-254_AE-6410-02A
- J3: value Conn_01x03 -> Molex_KK-254_AE-6410-03A
- J4, J5, J6: value Conn_01x02 Sub Osc Out -> Molex_KK-254_AE-6410-02A
- J7, J8: value Conn_01x01 -> Wire pad
Changed lines of the file:
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@@
       (effects (font (size 0.75 0.75) (thickness 0.15)))
     )
-    (fp_text value Conn_01x01 (at 0 3.175) (layer F.Fab)
+    (fp_text value "Wire pad" (at 0 3.175) (layer F.Fab)
       (effects (font (size 1 1) (thickness 0.15)))
     )
@@
       (effects (font (size 0.75 0.75) (thickness 0.15)))
     )
-    (fp_text value Conn_01x01 (at 0 3.175) (layer F.Fab)
+    (fp_text value "Wire pad" (at 0 3.175) (layer F.Fab)
       (effects (font (size 1 1) (thickness 0.15)))
     )
@@
       (effects (font (size 0.75 0.75) (thickness 0.15)))
     )
-    (fp_text value "Conn_01x02 Sub Osc Out" (at 1.27 4.08 90) (layer F.Fab)
+    (fp_text value Molex_KK-254_AE-6410-02A (at 1.27 4.08 90) (layer F.Fab)
       (effects (font (size 1 1) (thickness 0.15)))
     )
@@
       (effects (font (size 0.75 0.75) (thickness 0.15)))
     )
-    (fp_text value "Conn_01x02 Sub Osc Out" (at 1.27 4.08 90) (layer F.Fab)
+    (fp_text value Molex_KK-254_AE-6410-02A (at 1.27 4.08 90) (layer F.Fab)
       (effects (font (size 1 1) (thickness 0.15)))
     )
@@
       (effects (font (size 0.75 0.75) (thickness 0.15)))
     )
-    (fp_text value "Conn_01x02 Sub Osc Out" (at 1.27 4.08 90) (layer F.Fab)
+    (fp_text value Molex_KK-254_AE-6410-02A (at 1.27 4.08 90) (layer F.Fab)
       (effects (font (size 1 1) (thickness 0.15)))
     )
@@
       (effects (font (size 0.75 0.75) (thickness 0.15)))
     )
-    (fp_text value Conn_01x03 (at 2.54 4.08 90) (layer F.Fab)
+    (fp_text value Molex_KK-254_AE-6410-03A (at 2.54 4.08 90) (layer F.Fab)
       (effects (font (size 1 1) (thickness 0.15)))
     )
@@
       (effects (font (size 0.75 0.75) (thickness 0.15)))
     )
-    (fp_text value "Conn_01x02 Osc In" (at 1.27 4.08 90) (layer F.Fab)
-      (effects (font (size 1 1) (thickness 0.15)))
-    )
+    (fp_text value Molex_KK-254_AE-6410-02A (at 1.27 4.08 90) (layer F.Fab)
+      (effects (font (size 1 1) (thickness 0.15)))
+    )

Commit message: Comments in schematic and README
Connections:
- net /-1_OCT_1 renamed /-1_OCT
- net /-2_OCT_1 renamed /-2_OCT

Commit message: Schematic pdf, footprint, and 10nF, 10uF, what's the difference?
Other:
- board text added: "Omit from 2nd board"
- board text added: "Omit from both boards"

Commit message: Correct C1
Parts:
- C1: value 10uF -> 10nF; footprint ao_tht:CP_Radial_D5.0mm_P2.00mm -> ao_tht:C_Rect_L7.2mm_W2.5mm_P5.00mm_FKS2_FKP2_MKS2_MKP2
- C2: value 10uF -> 10uF (*)
- D2: value 1n5817 -> 1n5817 (*)
- D3, D4: value 1n4733 -> 1n4733 (*)
- J1, J5: value Molex_KK-254_AE-6410-02A -> 2 PIN HDR
- J2: value EURO_PWR_2x5 -> EURO_PWR_2x5 (*)
- J3: value Molex_KK-254_AE-6410-03A -> 3 PIN HDR
- J4, J6: value Molex_KK-254_AE-6410-02A -> 2 PIN HDR (*)
- R6, R7: value 1k -> 1k (*)
- moved C1 0.71 mm to (158.5, 81.5)
- moved U1 0.06 mm to (145.0, 73.1)
Connections:
- net CLOCK_DIV_2_OUT renamed Net-(D3-Pad1)
- net CLOCK_DIV_4_OUT renamed Net-(D4-Pad1)
- net OSC_INPUT renamed Net-(J1-Pad1)
- net SUB_OSC_OUT renamed Net-(D5-Pad2)
- U1 pad 4: GND -> Net-(U1-Pad4)
Routing:
- net Net-(C1-Pad1): track 20.2 -> 19.2 mm
